Commit message: update 311025

File: myrobot/urdf/myrobot_base.xacro (robot description, xacro)
@@ -1,5 +1,7 @@
 <?xml version="1.0"?>
 <robot name="Cuong_MobileRobot" xmlns:xacro="http://www.ros.org/wiki/xacro" >
-  <!-- BASE LINK -->
+  <xacro:property name="frame_ground_offset" value="0.02"/>
+  <xacro:property name="diff_wheels_radius" value="0.0501"/>
+<!-- Footprint link -->
   <link name="base_footprint">
   </link>
@@ -9,12 +11,16 @@
     <child link="base_link" />
   </joint>
-  <!-- Chassis LINK -->
+<!-- Base link -->
   <link name="base_link">
-   <inertial>
-      <origin
-        xyz="-0.00887608577321029 7.15767558960218E-06 0.0787840514491733"
-        rpy="0 0 0" />
-      <mass
-        value="1.28133453331002" />
+    <visual>
+      <origin xyz="0 0 ${frame_ground_offset}" rpy="0 0 0" />
+      <geometry>
+        <mesh filename="file://$(find myrobot)/meshes//base_link.STL" />
+      </geometry>
+      <material name="gray"/>
+    </visual>
+    <inertial>
+      <origin xyz="-0.0089 0 ${frame_ground_offset + 0.0788}" rpy="0 0 0" />
+      <mass value="1.281" />
       <inertia
         ixx="0.0468244369690289"
@@ -25,32 +31,26 @@
         izz="0.0664423696630811" />
     </inertial>
+    <collision>
+      <origin xyz="0 0 ${frame_ground_offset}" rpy="0 0 0" />
+      <geometry>
+        <mesh filename="file://$(find myrobot)/meshes//base_link.STL" />
+      </geometry>
+    </collision>
+  </link>
+<!-- Right-Drive link -->
+  <link name="RD_link">
     <visual>
       <origin
         xyz="0 0 0"
-        rpy="0 0 0" />
+        rpy="0 0 0"/>
       <geometry>
         <mesh
-          filename="file://$(find myrobot)/meshes//base_link.STL" />
-      </geometry>
-      <material name="gray"/>
-    </visual>
-    <collision>
-      <origin
-        xyz="0 0 0"
-        rpy="0 0 0" />
-      <geometry>
-        <mesh
-          filename="file://$(find myrobot)/meshes//base_link.STL" />
-      </geometry>
-    </collision>
-  </link>
-  <!-- RightDrive_link -->
-  <link name="RD_link">
-    <inertial>
-      <origin
-        xyz="7.87594729263556E-06 3.21954041912487E-07 -0.00125132754173546"
-        rpy="0 0 0" />
-      <mass
-        value="0.268087345954588" />
+          filename="file://$(find myrobot)/meshes//RD_link.STL" />
+      </geometry>
+      <material name="white"/>
+    </visual>
+    <inertial>
+      <origin xyz="0 0 0" rpy="0 0 0" />
+      <mass value="0.2681" />
       <inertia
         ixx="0.0001926951796097"
@@ -61,21 +61,8 @@
         izz="0.00032009896690558" />
     </inertial>
-    <visual>
-      <origin
-        xyz="0 0 0"
-        rpy="0 0 0" />
-      <geometry>
-        <mesh
-          filename="file://$(find myrobot)/meshes//RD_link.STL" />
-      </geometry>
-      <material name="white"/>
-    </visual>
-    <collision>
-      <origin
-        xyz="0 0 0"
-        rpy="0 0 0" />
-      <geometry>
-        <mesh
-          filename="file://$(find myrobot)/meshes//RD_link.STL" />
+    <collision>
+      <origin xyz="0 0 0" rpy="0 0 0" />
+      <geometry>
+            <sphere radius="${diff_wheels_radius}"/>
       </geometry>
     </collision>
@@ -83,17 +70,21 @@
   <joint name="RD_joint"
     type="continuous">
-    <origin xyz="0 -0.2014 0.03" rpy="1.5707963267949 0 0" />
+    <origin xyz="0 -0.2014 ${frame_ground_offset + 0.03}" rpy="${pi/2} 0 0" />
     <parent link="base_link" />
     <child link="RD_link" />
-    <axis xyz="0 0 1" />
-  </joint>
-  <!-- LeftDrive_link -->
+    <axis xyz="0 0 -1" />
+  </joint>
+<!-- Left-Drive link -->
   <link name="LD_link">
-    <inertial>
-      <origin
-        xyz="-3.79337303156049E-06 -6.90974103747036E-06 0.00125132754173543"
-        rpy="0 0 0" />
-      <mass
-        value="0.268087345954588" />
+    <visual>
+      <origin xyz="0 0 0" rpy="0 0 0" />
+      <geometry>
+        <mesh filename="file://$(find myrobot)/meshes//LD_link.STL" />
+      </geometry>
+      <material name="white"/>
+    </visual>
+    <inertial>
+      <origin xyz="0 0 0" rpy="0 0 0"/>C
+      <mass value="0.2681" />
       <inertia
         ixx="0.000192680084553262"
@@ -104,165 +95,109 @@
         izz="0.00032009896690558" />
     </inertial>
-    <visual>
-      <origin
-        xyz="0 0 0"
-        rpy="0 0 0" />
-      <geometry>
-        <mesh
-          filename="file://$(find myrobot)/meshes//LD_link.STL" />
-      </geometry>
-      <material name="white"/>
-    </visual>
-    <collision>
-      <origin
-        xyz="0 0 0"
-        rpy="0 0 0" />
-      <geometry>
-        <mesh
-          filename="file://$(find myrobot)/meshes//LD_link.STL" />
-      </geometry>
-    </collision>
+    <collision>
+      <origin xyz="0 0 0" rpy="0 0 0" />
+      <geometry>
+            <sphere radius="${diff_wheels_radius}"/>
+      </geometry>
+      </collision>
   </link>
   <joint name="LD_joint"
     type="continuous">
-    <origin
-      xyz="0 0.2014 0.03"
-      rpy="1.5707963267949 0 0" />
-    <parent
-      link="base_link" />
-    <child
-      link="LD_link" />
-    <axis
-      xyz="0 0 -1" />
-  </joint>
-  <!-- BackRightCaster_link -->
+    <origin xyz="0 0.2014 ${frame_ground_offset + 0.03}" rpy="${pi/2} 0 0" />
+    <parent link="base_link" />
+    <child link="LD_link" />
+    <axis xyz="0 0 -1" />
+  </joint>
+<!-- Caster links -->
+  <!-- Back-Right-Caster link -->
   <link name="BRC_link">
-    <inertial>
-      <origin
-        xyz="0.00480643793588634 0.00813240295364562 5.61462762532772E-08"
-        rpy="0 0 0" />
-      <mass
-        value="0.028455048288764" />
-      <inertia
-        ixx="3.94774719095158E-06"
-        ixy="-2.92353662392493E-07"
-        ixz="-7.18479870958837E-11"
-        iyy="4.24152605662568E-06"
-        iyz="-8.83598650868593E-12"
-        izz="5.71387977555985E-06" />
-    </inertial>
-    <visual>
-      <origin
-        xyz="0 0 0"
-        rpy="0 0 0" />
-      <geometry>
-        <mesh
-          filename="file://$(find myrobot)/meshes//BRC_link.STL" />
-      </geometry>
-      <material name="white"/>
-    </visual>
-    <collision>
-      <origin
-        xyz="0 0 0"
-        rpy="0 0 0" />
-      <geometry>
-        <mesh
-          filename="file://$(find myrobot)/meshes//BRC_link.STL" />
-      </geometry>
-    </collision>
-  </link>
-  <joint name="BRC_joint"
-    type="fixed">
-    <origin
-      xyz="-0.166647236505441 -0.12 0"
-      rpy="1.5707963267949 0 0" />
-    <parent
-      link="base_link" />
-    <child
-      link="BRC_link" />
-    <axis
-      xyz="0 0 0" />
-  </joint>
-  <!-- BackLeftCaster_link -->
+    <visual>
+      <origin xyz="0 0 0" rpy="0 0 0" />
+      <geometry>
+        <mesh filename="file://$(find myrobot)/meshes//BRC_link.STL" />
+      </geometry>
+      <material name="white"/>
+    </visual>
+    <inertial>
+      <origin xyz="0.0048 0.0081 0" rpy="0 0 0"/>
+      <mass value="0.0284"/>
+      <inertia
+        ixx="3.94774719095158E-06"
+        ixy="-2.92353662392493E-07"
+        ixz="-7.18479870958837E-11"
+        iyy="4.24152605662568E-06"
+        iyz="-8.83598650868593E-12"
+        izz="5.71387977555985E-06"/>
+    </inertial>
+    <collision>
+      <origin xyz="0 0 0" rpy="0 0 0" />
+      <geometry>
+        <mesh filename="file://$(find myrobot)/meshes//BRC_link.STL" />
+      </geometry>
+    </collision>
+  </link>
+  <joint name="BRC_joint" type="fixed">
+    <origin xyz="-0.1666 -0.12 ${frame_ground_offset}" rpy="${pi/2} 0 0" />
+    <parent link="base_link" />
+    <child link="BRC_link" />
+    <axis xyz="0 0 0" />
+  </joint>
+  <!-- Back-Left-Caster link -->
   <link name="BLC_link">
-    <inertial>
-      <origin
-        xyz="0.00480643793588639 0.00813240295364563 5.61462762393994E-08"
-        rpy="0 0 0" />
-      <mass
-        value="0.0284550482887641" />
-      <inertia
-        ixx="3.9477471909516E-06"
-        ixy="-2.92353662392497E-07"
-        ixz="-7.18479870979925E-11"
-        iyy="4.24152605662568E-06"
-        iyz="-8.83598650523835E-12"
-        izz="5.71387977555987E-06" />
-    </inertial>
-    <visual>
-      <origin
-        xyz="0 0 0"
-        rpy="0 0 0" />
-      <geometry>
-        <mesh
-          filename="file://$(find myrobot)/meshes//BLC_link.STL" />
-      </geometry>
-      <material name="white"/>
-    </visual>
-    <collision>
-      <origin
-        xyz="0 0 0"
-        rpy="0 0 0" />
-      <geometry>
-        <mesh
-          filename="file://$(find myrobot)/meshes//BLC_link.STL" />
-      </geometry>
-    </collision>
-  </link>
-  <joint name="BLC_joint"
-    type="fixed">
-    <origin
-      xyz="-0.166647236505441 0.12 0"
-      rpy="1.5707963267949 0 0" />
-    <parent
-      link="base_link" />
-    <child
-      link="BLC_link" />
-    <axis
-      xyz="0 0 0" />
-  </joint>
-  <!-- FrontRightCaster_link -->
+    <visual>
+      <origin xyz="0 0 0" rpy="0 0 0" />
+      <geometry>
+        <mesh filename="file://$(find myrobot)/meshes//BLC_link.STL" />
+      </geometry>
+      <material name="white"/>
+    </visual>
+    <inertial>
+      <origin xyz="0.0048 0.0081 0" rpy="0 0 0"/>
+      <mass value="0.0284"/>
+      <inertia
+        ixx="3.94774719095158E-06"
+        ixy="-2.92353662392493E-07"
+        ixz="-7.18479870958837E-11"
+        iyy="4.24152605662568E-06"
+        iyz="-8.83598650868593E-12"
+        izz="5.71387977555985E-06"/>
+    </inertial>
+    <collision>
+      <origin xyz="0 0 0" rpy="0 0 0" />
+      <geometry>
+        <mesh filename="file://$(find myrobot)/meshes//BLC_link.STL" />
+      </geometry>
+    </collision>
+  </link>
+  <joint name="BLC_joint" type="fixed">
+    <origin xyz="-0.1666 0.12 ${frame_ground_offset}" rpy="${pi/2} 0 0" />
+    <parent link="base_link" />
+    <child link="BLC_link" />
+    <axis xyz="0 0 0" />
+  </joint>
+  <!-- Front-Right-Caster link -->
   <link name="FRC_link">
-    <inertial>
-      <origin
-        xyz="0.00480643793588634 0.00813240295364561 5.61462762255216E-08"
-        rpy="0 0 0" />
-      <mass
-        value="0.028455048288764" />
-      <inertia
-        ixx="3.94774719095158E-06"
-        ixy="-2.92353662392493E-07"
-        ixz="-7.1847987094674E-11"
-        iyy="4.24152605662568E-06"
-        iyz="-8.83598650915944E-12"
-        izz="5.71387977555985E-06" />
-    </inertial>
-    <visual>
-      <origin
-        xyz="0 0 0"
-        rpy="0 0 0" />
-      <geometry>
-        <mesh
-          filename="file://$(find myrobot)/meshes//FRC_link.STL" />
-      </geometry>
-      <material name="white"/>
-    </visual>
-    <collision>
-      <origin
-        xyz="0 0 0"
-        rpy="0 0 0" />
-      <geometry>
-        <mesh
-          filename="file://$(find myrobot)/meshes//FRC_link.STL" />
+    <visual>
+      <origin xyz="0 0 0" rpy="0 0 0" />
+      <geometry>
+        <mesh filename="file://$(find myrobot)/meshes//FRC_link.STL" />
+      </geometry>
+      <material name="white"/>
+    </visual>
+    <inertial>
+      <origin xyz="0.0048 0.0081 0" rpy="0 0 0"/>
+      <mass value="0.0284"/>
+      <inertia
+        ixx="3.94774719095158E-06"
+        ixy="-2.92353662392493E-07"
+        ixz="-7.18479870958837E-11"
+        iyy="4.24152605662568E-06"
+        iyz="-8.83598650868593E-12"
+        izz="5.71387977555985E-06"/>
+    </inertial>
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
File: myrobot/urdf/myrobot_gazebo.xacro (robot description, xacro)
@@ -48,5 +48,5 @@
             <left_joint>LD_joint</left_joint>
             <right_joint>RD_joint</right_joint>
-            <wheel_separation>0.5</wheel_separation>
+            <wheel_separation>0.4</wheel_separation>
             <wheel_diameter>0.1</wheel_diameter>
             <max_wheel_torque>96.25</max_wheel_torque>
